File: hardware/SparkFun_Pi_Wedge_40-Pin_PreAssembled.sch (EAGLE design)
At the start: 17 parts

Commit message: Updates after group review.
A few silk touch-ups.
Renaming to "Pi Wedge 40-Pin".
Other:
- note added: "V10"
- note removed: "V01"
Changed lines of the file:
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@@
 <plain>
 <text x="172.72" y="10.16" size="2.54" layer="94" font="vector">Byron Jacquot</text>
-<text x="238.76" y="7.62" size="2.54" layer="94" font="vector">V01</text>
+<text x="238.76" y="7.62" size="2.54" layer="94" font="vector">V10</text>
 <text x="114.3" y="48.26" size="2.54" layer="94" font="vector">All logic signals are 3.3V, and not 5V tolerant.
 There is no over-voltage protection on the RPi, nor

Commit message: Updates after checklist review.
Parts:
- JP2: value RASPBERRYPI-B+-GPIO-SMT -> RASPBERRYPI-40-PIN-GPIO-SMT; device SparkFun-Boards:RASPBERRYPI-B+-GPIO-SMT -> SparkFun-Boards:RASPBERRYPI-40-PIN-GPIO-SMT
Other:
- note added: "All logic signals are 3.3V, and not 5V tolerant. There is no over-voltage protection on the RPi, nor on the Pi Wedge."
- note removed: "All logic signals are 3.3V, and not 5V tolerant. There is no over-voltage protection on the RPi, nor on the Pi Wedge B+."
Changed lines of the file:
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@@
 <part name="SUPPLY10" library="SparkFun-Aesthetics" deviceset="3.3V" device=""/>
 <part name="U$2" library="SparkFun-Aesthetics" deviceset="BREADBOARD_PATTERN" device=""/>
-<part name="JP2" library="SparkFun-Boards" deviceset="RASPBERRYPI-B+-GPIO" device="-SMT" value="RASPBERRYPI-B+-GPIO-SMT"/>
+<part name="JP2" library="SparkFun-Boards" deviceset="RASPBERRYPI-40-PIN-GPIO" device="-SMT" value="RASPBERRYPI-40-PIN-GPIO-SMT"/>
 <part name="JP3" library="SparkFun-Connectors" deviceset="M17" device="KIT" value="1x17"/>
 <part name="JP4" library="SparkFun-Connectors" deviceset="M17" device="KIT" value="1x17"/>
@@
 <text x="114.3" y="48.26" size="2.54" layer="94" font="vector">All logic signals are 3.3V, and not 5V tolerant.
 There is no over-voltage protection on the RPi, nor
-on the Pi Wedge B+.</text>
+on the Pi Wedge.</text>
 <text x="7.62" y="50.8" size="2.54" layer="94" font="vector">TXO and RXI use 3.3V logic levels.
 Use with 3.3V FTDI adapter.</text>

Commit message: Updating caps values.
It had 47uf library parts (CAP-10547), but the schem incorrectly showed
10uf as the value.

Schem now reads 47uf.
Parts:
- C3V, C5V: value 10uf -> 47uf
Changed lines of the file:
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@@
 <part name="STANDOFF1" library="SparkFun-Electromechanical" deviceset="STAND-OFF" device=""/>
 <part name="STANDOFF2" library="SparkFun-Electromechanical" deviceset="STAND-OFF" device=""/>
-<part name="C5V" library="SparkFun-Capacitors" deviceset="47UF-50V-20%(ELECT)" device="" value="10uf"/>
-<part name="C3V" library="SparkFun-Capacitors" deviceset="47UF-50V-20%(ELECT)" device="" value="10uf"/>
+<part name="C5V" library="SparkFun-Capacitors" deviceset="47UF-50V-20%(ELECT)" device="" value="47uf"/>
+<part name="C3V" library="SparkFun-Capacitors" deviceset="47UF-50V-20%(ELECT)" device="" value="47uf"/>
 <part name="GND4" library="SparkFun" deviceset="GND" device=""/>
 <part name="GND8" library="SparkFun" deviceset="GND" device=""/>
